Commit message: colorize ur10

File: ur10e/ur10e.urdf (robot description, URDF)
Before this commit: robot ur10e, 12 links, 11 joints
Links:
- added link base1, mass 0.0; visual mesh filename=visual/base1.dae
- added link forearm2, mass 0.0; visual mesh filename=visual/forearm2.dae
- added link forearm3, mass 0.0; visual mesh filename=visual/forearm3.dae
- added link forearm4, mass 0.0; visual mesh filename=visual/forearm4.dae
- added link forearm5, mass 0.0; visual mesh filename=visual/forearm5.dae
- added link forearm6, mass 0.0; visual mesh filename=visual/forearm6.dae
- added link forearm7, mass 0.0; visual mesh filename=visual/forearm7.dae
- added link shoulder2, mass 0.0; visual mesh filename=visual/shoulder2.dae
- added link shoulder3, mass 0.0; visual mesh filename=visual/shoulder3.dae
- added link upperarm2, mass 0.0; visual mesh filename=visual/upperarm2.dae
- added link upperarm3, mass 0.0; visual mesh filename=visual/upperarm3.dae
- added link upperarm4, mass 0.0; visual mesh filename=visual/upperarm4.dae
- added link upperarm5, mass 0.0; visual mesh filename=visual/upperarm5.dae
- added link upperarm6, mass 0.0; visual mesh filename=visual/upperarm6.dae
- added link upperarm7, mass 0.0; visual mesh filename=visual/upperarm7.dae
- added link upperarm8, mass 0.0; visual mesh filename=visual/upperarm8.dae
- added link wrist_1_2, mass 0.0; visual mesh filename=visual/wrist1_2.dae
- added link wrist_1_3, mass 0.0; visual mesh filename=visual/wrist1_3.dae
- added link wrist_2_2, mass 0.0; visual mesh filename=visual/wrist2_2.dae
- added link wrist_2_3, mass 0.0; visual mesh filename=visual/wrist2_3.dae
- link base_link: geometry collision mesh filename=collision/base.stl; visual mesh filename=visual/base2.dae
- link forearm_link: geometry collision mesh filename=collision/forearm.stl; visual mesh filename=visual/forearm1.dae
- link shoulder_link: geometry collision mesh filename=collision/shoulder.stl; visual mesh filename=visual/shoulder1.dae
- link upper_arm_link: geometry collision mesh filename=collision/upperarm.stl; visual mesh filename=visual/upperarm1.dae
- link wrist_1_link: geometry collision mesh filename=collision/wrist1.stl; visual mesh filename=visual/wrist1_1.dae
- link wrist_2_link: geometry collision mesh filename=collision/wrist2.stl; visual mesh filename=visual/wrist2_1.dae
Joints:
- added joint base1-base_link_fixed_joint: type fixed, parent base1, child base_link, origin xyz=0 0 0 rpy=0 0 0
- added joint forearm_link-forearm2_fixed_joint: type fixed, parent forearm_link, child forearm2
- added joint forearm_link-forearm3_fixed_joint: type fixed, parent forearm_link, child forearm3
- added joint forearm_link-forearm4_fixed_joint: type fixed, parent forearm_link, child forearm4
- added joint forearm_link-forearm5_fixed_joint: type fixed, parent forearm_link, child forearm5
- added joint forearm_link-forearm6_fixed_joint: type fixed, parent forearm_link, child forearm6
- added joint forearm_link-forearm7_fixed_joint: type fixed, parent forearm_link, child forearm7
- added joint shoulder_link-shoulder2_fixed_joint: type fixed, parent shoulder_link, child shoulder2
- added joint shoulder_link-shoulder3_fixed_joint: type fixed, parent shoulder_link, child shoulder3
- added joint upper_arm_link-upperarm2_fixed_joint: type fixed, parent upper_arm_link, child upperarm2
- added joint upper_arm_link-upperarm3_fixed_joint: type fixed, parent upper_arm_link, child upperarm3
- added joint upper_arm_link-upperarm4_fixed_joint: type fixed, parent upper_arm_link, child upperarm4
- added joint upper_arm_link-upperarm5_fixed_joint: type fixed, parent upper_arm_link, child upperarm5
- added joint upper_arm_link-upperarm6_fixed_joint: type fixed, parent upper_arm_link, child upperarm6
- added joint upper_arm_link-upperarm7_fixed_joint: type fixed, parent upper_arm_link, child upperarm7
- added joint upper_arm_link-upperarm8_fixed_joint: type fixed, parent upper_arm_link, child upperarm8
- added joint wrist_1_link-wrist_1_2_fixed_joint: type fixed, parent wrist_1_link, child wrist_1_2
- added joint wrist_1_link-wrist_1_3_fixed_joint: type fixed, parent wrist_1_link, child wrist_1_3
- added joint wrist_2_link-wrist_2_2_fixed_joint: type fixed, parent wrist_2_link, child wrist_2_2
- added joint wrist_2_link-wrist_2_3_fixed_joint: type fixed, parent wrist_2_link, child wrist_2_3
